Commit message: Use all STL's in simple URDF (+base/pedestal)
Changes the remaining DAE files to STL's for the baxter_simple.urdf
This allows STL parsers like RViz for Android to visualize them.
There should probably be simplified textures for these last three
STL's created too.

File: baxter_description/urdf/baxter_simple.urdf (robot description, URDF)
Before this commit: robot baxter, 49 links, 48 joints
Links:
- link torso: geometry collision mesh filename=package://baxter_description/meshes/torso/base_link_collisi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; visual mesh filename=package://baxter_description/meshes/torso/base_link.STL

Commit message: use collision stl for simple_baxter.urdf

File: baxter_description/urdf/baxter_simple.urdf (robot description, URDF)
Before this commit: robot baxter, 49 links, 48 joints
Links:
- link pedestal: geometry collision mesh filename=package://baxter_description/meshes/base/pedestal_link_coll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; visual mesh filename=package://baxter_description/meshes/base/pedestal_link_coll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
- link torso: geometry collision mesh filename=package://baxter_description/meshes/torso/base_link_collisi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; visual mesh filename=package://baxter_description/meshes/torso/base_link_collisi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
