Commit message: Removing urdf gripper_base frames not yet reflected on robot.

File: baxter_description/urdf/baxter.urdf (robot description, URDF)
Before this commit: robot baxter, 46 links, 45 joints
Links:
- removed link left_gripper_base
- removed link right_gripper_base
- link base: mass 0.0001 -> 0.00094542
- link collision_head_link_1: mass 0.0001 -> 0.00094542
- link collision_head_link_2: mass 0.0001 -> 0.00094542
- link dummyhead1: mass 0.0001 -> 0.00094542
- link head_camera: mass 0.0001 -> 0.00094542
- link left_arm_itb: mass 0.0001 -> 0.00094542
- link left_arm_mount: mass 0.0001 -> 0.00094542
- link left_gripper: mass 0.0001 -> 0.00094542; geometry visual box size=0.025 0.075 0.035
- link left_hand_camera: mass 0.0001 -> 0.00094542
- link left_hand_camera_axis: mass 0.0001 -> 0.00094542
- link left_hand_range: mass 0.0001 -> 0.00094542
- link left_torso_itb: mass 0.0001 -> 0.00094542
- link left_upper_elbow_visual: mass 0.0001 -> 0.00094542
- link left_upper_forearm_visual: mass 0.0001 -> 0.00094542
- link right_arm_itb: mass 0.0001 -> 0.00094542
- link right_arm_mount: mass 0.0001 -> 0.00094542
- link right_gripper: mass 0.0001 -> 0.00094542; geometry visual box size=0.025 0.075 0.035
- link right_hand_camera: mass 0.0001 -> 0.00094542
- link right_hand_camera_axis: mass 0.0001 -> 0.00094542
- link right_hand_range: mass 0.0001 -> 0.00094542
- link right_torso_itb: mass 0.0001 -> 0.00094542
- link right_upper_elbow_visual: mass 0.0001 -> 0.00094542
- link right_upper_forearm_visual: mass 0.0001 -> 0.00094542
- link sonar_ring: mass 0.0001 -> 0.00094542
Joints:
- removed joint left_gripper_base
- removed joint right_gripper_base
- joint left_endpoint: parent left_gripper_base -> left_hand
- joint right_endpoint: parent right_gripper_base -> right_hand

Commit message: adding damping values to URDF. fixes #1.

File: baxter_description/urdf/baxter.urdf (robot description, URDF)
Before this commit: robot baxter, 44 links, 43 joints
Links:
- link head: geometry collision sphere radius=0.001; visual mesh filename=package://baxter_description/meshes/head/H0.STL
- link left_lower_elbow: geometry collision cylinder length=0.10 radius=0.06; visual mesh filename=package://baxter_description/meshes/lower_elbow/E1.STL
- link left_lower_forearm: geometry collision cylinder length=0.10 radius=0.06; visual mesh filename=package://baxter_description/meshes/lower_forearm/W1.STL
- link left_lower_shoulder: geometry collision cylinder length=0.12 radius=0.06; visual mesh filename=package://baxter_description/meshes/lower_shoulder/S1.STL
- link left_upper_elbow: geometry collision cylinder length=0.107 radius=0.06; visual mesh filename=package://baxter_description/meshes/upper_elbow/E0.STL
- link left_upper_forearm: geometry collision cylinder length=0.088 radius=0.06; visual mesh filename=package://baxter_description/meshes/upper_forearm/W0.STL
- link left_upper_shoulder: geometry collision cylinder length=0.2722 radius=0.06; visual mesh filename=package://baxter_description/meshes/upper_shoulder/S0.STL
- link left_wrist: geometry collision cylinder length=0.165 radius=0.06; visual mesh filename=package://baxter_description/meshes/wrist/W2.STL
- link pedestal: geometry collision box size=0.92 0.83 0.3; visual mesh filename=package://baxter_description/meshes/base/PEDESTAL.STL
- link right_lower_elbow: geometry collision cylinder length=0.10 radius=0.06; visual mesh filename=package://baxter_description/meshes/lower_elbow/E1.STL
- link right_lower_forearm: geometry collision cylinder length=0.10 radius=0.06; visual mesh filename=package://baxter_description/meshes/lower_forearm/W1.STL
- link right_lower_shoulder: geometry collision cylinder length=0.12 radius=0.06; visual mesh filename=package://baxter_description/meshes/lower_shoulder/S1.STL
- link right_upper_elbow: geometry collision cylinder length=0.107 radius=0.06; visual mesh filename=package://baxter_description/meshes/upper_elbow/E0.STL
- link right_upper_forearm: geometry collision cylinder length=0.088 radius=0.06; visual mesh filename=package://baxter_description/meshes/upper_forearm/W0.STL
- link right_upper_shoulder: geometry collision cylinder length=0.2722 radius=0.06; visual mesh filename=package://baxter_description/meshes/upper_shoulder/S0.STL
- link right_wrist: geometry collision cylinder length=0.165 radius=0.06; visual mesh filename=package://baxter_description/meshes/wrist/W2.STL
- link screen: geometry collision sphere radius=0.001; visual mesh filename=package://baxter_description/meshes/head/H1.STL
- link torso: geometry collision cylinder length=0.7 radius=0.27; visual mesh filename=package://baxter_description/meshes/torso/base_link.STL

Commit message: Respecifying DAEs in URDF.

File: baxter_description/urdf/baxter.urdf (robot description, URDF)
Before this commit: robot baxter, 44 links, 43 joints
Links:
- link head: geometry collision sphere radius=0.001; visual mesh filename=package://baxter_description/meshes/head/H0.DAE
- link left_lower_elbow: geometry collision cylinder length=0.10 radius=0.06; visual mesh filename=package://baxter_description/meshes/lower_elbow/E1.DAE
- link left_lower_forearm: geometry collision cylinder length=0.10 radius=0.06; visual mesh filename=package://baxter_description/meshes/lower_forearm/W1.DAE
- link left_lower_shoulder: geometry collision cylinder length=0.12 radius=0.06; visual mesh filename=package://baxter_description/meshes/lower_shoulder/S1.DAE
- link left_upper_elbow: geometry collision cylinder length=0.107 radius=0.06; visual mesh filename=package://baxter_description/meshes/upper_elbow/E0.DAE
- link left_upper_forearm: geometry collision cylinder length=0.088 radius=0.06; visual mesh filename=package://baxter_description/meshes/upper_forearm/W0.DAE
- link left_upper_shoulder: geometry collision cylinder length=0.2722 radius=0.06; visual mesh filename=package://baxter_description/meshes/upper_shoulder/S0.DAE
- link left_wrist: geometry collision cylinder length=0.165 radius=0.06; visual mesh filename=package://baxter_description/meshes/wrist/W2.DAE
- link pedestal: geometry collision box size=0.92 0.83 0.3; visual mesh filename=package://baxter_description/meshes/base/PEDESTAL.DAE
- link right_lower_elbow: geometry collision cylinder length=0.10 radius=0.06; visual mesh filename=package://baxter_description/meshes/lower_elbow/E1.DAE
- link right_lower_forearm: geometry collision cylinder length=0.10 radius=0.06; visual mesh filename=package://baxter_description/meshes/lower_forearm/W1.DAE
- link right_lower_shoulder: geometry collision cylinder length=0.12 radius=0.06; visual mesh filename=package://baxter_description/meshes/lower_shoulder/S1.DAE
- link right_upper_elbow: geometry collision cylinder length=0.107 radius=0.06; visual mesh filename=package://baxter_description/meshes/upper_elbow/E0.DAE
- link right_upper_forearm: geometry collision cylinder length=0.088 radius=0.06; visual mesh filename=package://baxter_description/meshes/upper_forearm/W0.DAE
- link right_upper_shoulder: geometry collision cylinder length=0.2722 radius=0.06; visual mesh filename=package://baxter_description/meshes/upper_shoulder/S0.DAE
- link right_wrist: geometry collision cylinder length=0.165 radius=0.06; visual mesh filename=package://baxter_description/meshes/wrist/W2.DAE
- link screen: geometry collision sphere radius=0.001; visual mesh filename=package://baxter_description/meshes/head/H1.DAE
- link torso: geometry collision cylinder length=0.7 radius=0.27; visual mesh filename=package://baxter_description/meshes/torso/base_link.DAE

Commit message: Fixed error 'The root link base has an inertia specified in the URDF, but KDL does not support a root link with an inertia.  As a workaround, you can add an extra dummy link to your URDF.'

File: baxter_description/urdf/baxter.urdf (robot description, URDF)
Before this commit: robot baxter, 44 links, 43 joints
Links:
- link base: mass 0.00094542 -> None

Commit message: Added screen visual display

File: baxter_description/urdf/baxter.urdf (robot description, URDF)
Before this commit: robot baxter, 44 links, 43 joints
Links:
- added link screen_visual, mass 0.001; visual box size=0.218 0.16 0.001
Joints:
- added joint screen_visual_joint: type fixed, parent screen, child screen_visual, origin xyz=0.0 -0.016 0.0 rpy=0 0 0

Commit message: Added updated base link for collisions

File: baxter_description/urdf/baxter.urdf (robot description, URDF)
Before this commit: robot baxter, 45 links, 44 joints
Links:
- link torso: geometry collision mesh filename=package://baxter_description/meshes/torso/base_link_collisi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; visual mesh filename=package://baxter_description/meshes/torso/base_link.DAE

Commit message: Updating Chris's pull for the low poly meshes per Dave's comment. Updating the urdf to reflect these new meshes.

File: baxter_description/urdf/baxter.urdf (robot description, URDF)
Before this commit: robot baxter, 45 links, 44 joints
Links:
- link base: geometry collision mesh filename=package://baxter_description/meshes/base/pedestal_link_coll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; visual mesh filename=package://baxter_description/meshes/base/PEDESTAL.DAE

Commit message: Updating pedestal collision dae.

File: baxter_description/urdf/baxter.urdf (robot description, URDF)
Before this commit: robot baxter, 45 links, 44 joints
Links:
- link base: geometry 
- link pedestal: geometry collision mesh filename=package://baxter_description/meshes/base/pedestal_link_coll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; visual mesh filename=package://baxter_description/meshes/base/PEDESTAL.DAE

Commit message: changes for 0.7 sdk

File: baxter_description/urdf/baxter.urdf (robot description, URDF)
Before this commit: robot baxter, 44 links, 43 joints
Links:
- link base: mass 0.00094542 -> None
- link pedestal: geometry collision mesh filename=package://baxter_description/meshes/base/pedestal_link_coll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; visual mesh filename=package://baxter_description/meshes/base/PEDESTAL.DAE
- link torso: geometry collision mesh filename=package://baxter_description/meshes/torso/base_link_collisi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; visual mesh filename=package://baxter_description/meshes/torso/base_link.DAE

Commit message: update urdf per latest robot side urdf

File: baxter_description/urdf/baxter.urdf (robot description, URDF)
Before this commit: robot baxter, 44 links, 43 joints
Links:
- added link left_gripper_base, mass 0.0001; visual box size=0.025 0.075 0.035
- added link right_gripper_base, mass 0.0001; visual box size=0.025 0.075 0.035
- link collision_head_link_1: mass 0.00094542 -> 0.0001
- link collision_head_link_2: mass 0.00094542 -> 0.0001
- link dummyhead1: mass 0.00094542 -> 0.0001
- link head_camera: mass 0.00094542 -> 0.0001
- link left_arm_itb: mass 0.00094542 -> 0.0001
- link left_arm_mount: mass 0.00094542 -> 0.0001
- link left_gripper: mass 0.00094542 -> 0.0001; geometry visual box size=0.01 0.01 0.01
- link left_hand_camera: mass 0.00094542 -> 0.0001
- link left_hand_camera_axis: mass 0.00094542 -> 0.0001
- link left_hand_range: mass 0.00094542 -> 0.0001
- link left_torso_itb: mass 0.00094542 -> 0.0001
- link left_upper_elbow_visual: mass 0.00094542 -> 0.0001
- link left_upper_forearm_visual: mass 0.00094542 -> 0.0001
- link right_arm_itb: mass 0.00094542 -> 0.0001
- link right_arm_mount: mass 0.00094542 -> 0.0001
- link right_gripper: mass 0.00094542 -> 0.0001; geometry visual box size=0.01 0.01 0.01
- link right_hand_camera: mass 0.00094542 -> 0.0001
- link right_hand_camera_axis: mass 0.00094542 -> 0.0001
- link right_hand_range: mass 0.00094542 -> 0.0001
- link right_torso_itb: mass 0.00094542 -> 0.0001
- link right_upper_elbow_visual: mass 0.00094542 -> 0.0001
- link right_upper_forearm_visual: mass 0.00094542 -> 0.0001
- link sonar_ring: mass 0.00094542 -> 0.0001
Joints:
- added joint left_gripper_base: type fixed, parent left_hand, child left_gripper_base, origin xyz=0 0 0 rpy=0 0 0
- added joint right_gripper_base: type fixed, parent right_hand, child right_gripper_base, origin xyz=0 0 0 rpy=0 0 0
- joint left_e0: limit lower=-3.05417993878 upper=3.05417993878 effort=60.0 velocity=2.5 -> lower=-3.05417993878 upper=3.05417993878 effort=50.0 velocity=1.5
- joint left_e1: limit lower=-0.05 upper=2.618 effort=60.0 velocity=2.5 -> lower=-0.05 upper=2.618 effort=50.0 velocity=1.5
- joint left_endpoint: origin xyz=0.0 0 0.05 rpy=0 0 0 -> xyz=0.0 0 0.025 rpy=0 0 0; parent left_hand -> left_gripper_base
- joint left_s0: limit lower=-1.70167993878 upper=1.70167993878 effort=60.0 velocity=2.5 -> lower=-1.70167993878 upper=1.70167993878 effort=50.0 velocity=1.5
- joint left_s1: limit lower=-2.147 upper=1.047 effort=60.0 velocity=2.5 -> lower=-2.147 upper=1.047 effort=50.0 velocity=1.5
- joint left_w0: limit lower=-3.059 upper=3.059 effort=20.0 velocity=5.0 -> lower=-3.059 upper=3.059 effort=15.0 velocity=4.0
- joint left_w1: limit lower=-1.57079632679 upper=2.094 effort=20.0 velocity=5.0 -> lower=-1.57079632679 upper=2.094 effort=15.0 velocity=4.0
- joint left_w2: limit lower=-3.059 upper=3.059 effort=20.0 velocity=5.0 -> lower=-3.059 upper=3.059 effort=15.0 velocity=4.0
- joint right_e0: limit lower=-3.05417993878 upper=3.05417993878 effort=60.0 velocity=2.5 -> lower=-3.05417993878 upper=3.05417993878 effort=50.0 velocity=1.5
- joint right_e1: limit lower=-0.05 upper=2.618 effort=60.0 velocity=2.5 -> lower=-0.05 upper=2.618 effort=50.0 velocity=1.5
- joint right_endpoint: origin xyz=0.0 0 0.05 rpy=0 0 0 -> xyz=0.0 0 0.025 rpy=0 0 0; parent right_hand -> right_gripper_base
- joint right_s0: limit lower=-1.70167993878 upper=1.70167993878 effort=60.0 velocity=2.5 -> lower=-1.70167993878 upper=1.70167993878 effort=50.0 velocity=1.5
- joint right_s1: limit lower=-2.147 upper=1.047 effort=60.0 velocity=2.5 -> lower=-2.147 upper=1.047 effort=50.0 velocity=1.5
- joint right_w0: limit lower=-3.059 upper=3.059 effort=20.0 velocity=5.0 -> lower=-3.059 upper=3.059 effort=15.0 velocity=4.0
- joint right_w1: limit lower=-1.57079632679 upper=2.094 effort=20.0 velocity=5.0 -> lower=-1.57079632679 upper=2.094 effort=15.0 velocity=4.0
- joint right_w2: limit lower=-3.059 upper=3.059 effort=20.0 velocity=5.0 -> lower=-3.059 upper=3.059 effort=15.0 velocity=4.0

Commit message: Synching robot urdf with latest head origin updates. Fixes urdf head origin frame location and screen tilt angle.

File: baxter_description/urdf/baxter.urdf (robot description, URDF)
Before this commit: robot baxter, 46 links, 45 joints
Joints:
- joint head_camera: origin xyz=0.12839 0.0 0.06368 rpy=1.9198622 0.0 1.57079632679 -> xyz=0.12839 0 0.06368 rpy=1.75057 0 1.57079632679
- joint head_nod: origin xyz=.088 0.0 0.0 rpy=1.9198622 0.0 1.57079632679 -> xyz=.1227 0 0 rpy=1.75057 0 1.57079632679
- joint head_pan: origin xyz=0.0947 0 0.686 rpy=0 0 0 -> xyz=0.06 0 0.686 rpy=0 0 0

Commit message: Modified the URDF to include the various sensor plugins

File: baxter_description/urdf/baxter.urdf (robot description, URDF)
Before this commit: robot baxter, 46 links, 45 joints
Links:
- added link display, mass 0.00094542; visual box size=0.218 0.16 0.001
Joints:
- added joint display_joint: type fixed, parent screen, child display, origin xyz=0.0 -0.016 0.0 rpy=0 0 0

Commit message: Adds accelerometer joints/links in support of Gazebo simulation
Cleans up/syncs with robot changes.

File: baxter_description/urdf/baxter.urdf (robot description, URDF)
Before this commit: robot baxter, 47 links, 46 joints
Links:
- added link left_hand_accelerometer, mass 0.0001; visual box size=0.01 0.01 0.01
- added link right_hand_accelerometer, mass 0.0001; visual box size=0.01 0.01 0.01
- link display: mass 0.00094542 -> 0.0001
Joints:
- added joint left_hand_accelerometer: type fixed, parent left_hand, child left_hand_accelerometer, origin xyz=0.00198 0.000133 -0.0146 rpy=0 0 0
- added joint right_hand_accelerometer: type fixed, parent right_hand, child right_hand_accelerometer, origin xyz=0.00198 0.000133 -0.0146 rpy=0 0 0

Commit message: The maximum effort for s1 joint is increased to 100

File: baxter_description/urdf/baxter.urdf (robot description, URDF)
Before this commit: robot baxter, 49 links, 48 joints
Joints:
- joint left_s1: limit lower=-2.147 upper=1.047 effort=50.0 velocity=1.5 -> lower=-2.147 upper=1.047 effort=100.0 velocity=1.5
- joint right_s1: limit lower=-2.147 upper=1.047 effort=50.0 velocity=1.5 -> lower=-2.147 upper=1.047 effort=100.0 velocity=1.5

Commit message: updated URDF to incorporate the indigo specific changes and fixed the base of the robot to the world

File: baxter_description/urdf/baxter.urdf (robot description, URDF)
Before this commit: robot baxter, 49 links, 48 joints
Links:
- added link world
Joints:
- added joint fixed: type fixed, parent world, child base

Commit message: update model with gripper

File: baxter_description/urdf/baxter.urdf (robot description, URDF)
Before this commit: robot baxter, 49 links, 48 joints
Links:
- added link left_gripper_l_finger, mass 0.00094542; collision mesh filename=package://baxter_description/meshes/electric_gripper/finger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; visual mesh filename=package://baxter_description/meshes/electric_gripper/finger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
- added link left_gripper_r_finger, mass 0.00094542; collision mesh filename=package://baxter_description/meshes/electric_gripper/finger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; visual mesh filename=package://baxter_description/meshes/electric_gripper/finger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
- added link right_gripper_l_finger, mass 0.00094542; collision mesh filename=package://baxter_description/meshes/electric_gripper/finger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; visual mesh filename=package://baxter_description/meshes/electric_gripper/finger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
- added link right_gripper_r_finger, mass 0.00094542; collision mesh filename=package://baxter_description/meshes/electric_gripper/finger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; visual mesh filename=package://baxter_description/meshes/electric_gripper/finger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
- link left_gripper_base: mass 0.0001 -> 0.00094542; geometry collision cylinder length=0.1 radius=0.0275; visual mesh filename=package://baxter_description/meshes/electric_gripper/electr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
- link right_gripper_base: mass 0.0001 -> 0.00094542; geometry collision cylinder length=0.1 radius=0.0275; visual mesh filename=package://baxter_description/meshes/electric_gripper/electr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
Joints:
- added joint left_gripper_l_finger_joint: type prismatic, parent left_gripper, child left_gripper_l_finger, origin xyz=0.0 0.06 0.035 rpy=0 0 0, axis 0 0 1, limit lower=-0.0125 upper=0.0095 effort=20.0 velocity=5.0
- added joint left_gripper_r_finger_joint: type prismatic, parent left_gripper, child left_gripper_r_finger, origin xyz=0.0 0.06 -0.035 rpy=0 0 0, axis 0 0 1, limit lower=-0.0125 upper=0.0095 effort=20.0 velocity=5.0, mimic joint=left_gripper_l_finger_joint multiplier=-1 offset=0
- added joint right_gripper_l_finger_joint: type prismatic, parent right_gripper, child right_gripper_l_finger, origin xyz=0.0 0.06 0.035 rpy=0 0 0, axis 0 0 1, limit lower=-0.0125 upper=0.0095 effort=20.0 velocity=5.0
- added joint right_gripper_r_finger_joint: type prismatic, parent right_gripper, child right_gripper_r_finger, origin xyz=0.0 0.06 -0.035 rpy=0 0 0, axis 0 0 1, limit lower=-0.0125 upper=0.0095 effort=20.0 velocity=5.0, mimic joint=right_gripper_l_finger_joint multiplier=-1 offset=0
- joint left_endpoint: origin xyz=0.0 0 0.025 rpy=0 0 0 -> xyz=-0.005 0.0 0.02 rpy=1.57 0 0; parent left_gripper_base -> left_hand
- joint right_endpoint: origin xyz=0.0 0 0.025 rpy=0 0 0 -> xyz=-0.005 0.0 0.02 rpy=1.57 0 0; parent right_gripper_base -> right_hand

Commit message: model with gripper for development

File: baxter_description/urdf/baxter.urdf (robot description, URDF)
Before this commit: robot baxter, 49 links, 48 joints
Links:
- added link left_gripper_l_finger, mass 0.01; collision mesh filename=package://baxter_description/meshes/electric_gripper/finger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; visual mesh filename=package://baxter_description/meshes/electric_gripper/finger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
- added link left_gripper_r_finger, mass 0.01; collision mesh filename=package://baxter_description/meshes/electric_gripper/finger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; visual mesh filename=package://baxter_description/meshes/electric_gripper/finger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
- added link right_gripper_l_finger, mass 0.01; collision mesh filename=package://baxter_description/meshes/electric_gripper/finger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; visual mesh filename=package://baxter_description/meshes/electric_gripper/finger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
- added link right_gripper_r_finger, mass 0.01; collision mesh filename=package://baxter_description/meshes/electric_gripper/finger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; visual mesh filename=package://baxter_description/meshes/electric_gripper/finger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
- link left_gripper_base: mass 0.0001 -> 0.00094542; geometry collision cylinder length=0.1 radius=0.0275; visual mesh filename=package://baxter_description/meshes/electric_gripper/electr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
- link right_gripper_base: mass 0.0001 -> 0.00094542; geometry collision cylinder length=0.1 radius=0.0275; visual mesh filename=package://baxter_description/meshes/electric_gripper/electr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
Joints:
- added joint l_gripper_l_finger_joint: type prismatic, parent left_gripper, child left_gripper_l_finger, origin xyz=0.0 0.06 0.035 rpy=0 0 0, axis 0 0 1, limit lower=-0.0215 upper=0.0095 effort=20.0 velocity=5.0, mimic joint=l_gripper_r_finger_joint multiplier=-1 offset=0
- added joint l_gripper_r_finger_joint: type prismatic, parent left_gripper, child left_gripper_r_finger, origin xyz=0.0 0.06 -0.035 rpy=0 0 0, axis 0 0 1, limit lower=-0.0095 upper=0.0215 effort=20.0 velocity=5.0
- added joint r_gripper_l_finger_joint: type prismatic, parent right_gripper, child right_gripper_l_finger, origin xyz=0.0 0.06 0.035 rpy=0 0 0, axis 0 0 1, limit lower=-0.0215 upper=0.0095 effort=20.0 velocity=5.0, mimic joint=r_gripper_r_finger_joint multiplier=-1 offset=0
- added joint r_gripper_r_finger_joint: type prismatic, parent right_gripper, child right_gripper_r_finger, origin xyz=0.0 0.06 -0.035 rpy=0 0 0, axis 0 0 1, limit lower=-0.0095 upper=0.0215 effort=20.0 velocity=5.0
- joint left_endpoint: origin xyz=0.0 0 0.025 rpy=0 0 0 -> xyz=-0.005 0.0 0.02 rpy=1.57 0 0; parent left_gripper_base -> left_hand
- joint right_endpoint: origin xyz=0.0 0 0.025 rpy=0 0 0 -> xyz=-0.005 0.0 0.02 rpy=1.57 0 0; parent right_gripper_base -> right_hand
