Commit message: Added Xacro Infra for Dynamic Grippers Constructs
- Rotated the long_narrow finger dae (for testing, will delete in future)
- Rotated and translated the paddle_tip dae so that the origin
  corresponds with the finger's tip. This should be standard for all
  finger tips in the future
- Added new xacro files corresponding to fingers and tips of fingers.
  Every new finger and tip will get its own xacro. This allows us to
  control the mass, rotation, and translation between different fingers
- Improved the baxter_electric_gripper.xacro to ask for intuitive
  descriptions of the electric gripper, such as finger mount points,
  finger and finger tip
- Removed the dependance on baxter.urdf.xacro - our base URDF will
  always be baxter.urdf to preserve backwards compatibility

File: baxter_description/urdf/baxter_electric_gripper.urdf.xacro (robot description, xacro)
@@ -1,7 +1,8 @@
 <?xml version="1.0"?>
-<robot xmlns:xacro="http://www.ros.org/wiki/xacro" name="baxter_with_rethink_electric_gripper">
-  <xacro:include filename="$(find baxter_description)/urdf/baxter_base.xacro" />
+<robot xmlns:xacro="http://www.ros.org/wiki/xacro" name="baxter">
+  <xacro:include filename="$(find baxter_description)/urdf/baxter.urdf" />
   <xacro:include filename="$(find baxter_description)/urdf/rethink_electric_gripper.xacro" />
-  <xacro:rethink_electric_gripper side="right" gripper_side="r"/>
-  <xacro:rethink_electric_gripper side="left"  gripper_side="l"/>
+  <xacro:rethink_electric_gripper side="left" gripper_side="l" l_finger="extended_narrow" l_finger_slot="1" add_l_finger_tip="true" l_finger_tip="paddle_tip" r_finger="extended_narrow" r_finger_slot="1" add_r_finger_tip="true" r_finger_tip="paddle_tip"/>
+  <xacro:rethink_electric_gripper side="right" gripper_side="r" l_finger="extended_narrow" l_finger_slot="1" add_l_finger_tip="false" l_finger_tip="false" r_finger="extended_narrow" r_finger_slot="1" add_r_finger_tip="false" r_finger_tip="false"/>
+  <!-- basic_hard_tip -->
 </robot>

File: baxter_description/urdf/rethink_electric_gripper.xacro (robot description, xacro)
@@ -1,10 +1,11 @@
 <?xml version="1.0"?>
 <robot xmlns:xacro="http://www.ros.org/wiki/xacro" name="rethink_electric_gripper">
-  <xacro:macro name="rethink_electric_gripper" params="side gripper_side">
+  <xacro:property name="pi" value="3.1415926535897931" />
+  <xacro:macro name="rethink_electric_gripper" params="side gripper_side  r_finger r_finger_slot add_r_finger_tip r_finger_tip l_finger l_finger_slot add_l_finger_tip l_finger_tip">
     <!-- Base of end effector -->
-    <link name="${side}_gripper_base">
+    <link name="${side}_gripper_electric_base">
       <gravity>0</gravity>
       <visual>
-        <origin rpy="-1.57079632679 3.1415 0" xyz="0.00 0.00 0.025"/>
+        <origin rpy="${-pi/2} ${pi} 0" xyz="0 0 0"/>
         <geometry>
           <mesh filename="package://baxter_description/meshes/electric_gripper/electric_gripper_base.DAE"/>
@@ -12,7 +13,7 @@
       </visual>
       <collision>
-        <origin rpy="0 0 0" xyz="0.007 0.007 0"/>
+        <origin rpy="${-pi/2} ${pi} 0" xyz="0.0 0.0 0"/>
         <geometry>
-          <cylinder length="0.1" radius="0.0275"/>
+          <cylinder length="0.1" radius="0.029"/>
         </geometry>
         <material name="darkred">
@@ -21,104 +22,38 @@
       </collision>
       <inertial>
-        <origin rpy="0 0 0" xyz="0.000000 0.000000 0.000000"/>
-        <mass value="0.00094542"/>
+        <origin rpy="${-pi/2} ${pi} 0" xyz="0.0 0.0 0.0"/>
+        <mass value="0.3"/>
         <inertia ixx="2e-08" ixy="0" ixz="0" iyy="3e-08" iyz="0" izz="2e-08"/>
       </inertial>
     </link>
-    <link name="${side}_gripper">
-      <gravity>0</gravity>
-      <visual>
-        <origin rpy="0 0 0" xyz="0 0 0"/>
-        <geometry>
-          <box size="0.01 0.01 0.01"/>
-        </geometry>
-        <material name="rblack">
-          <color rgba="0 0 0 1"/>
-        </material>
-      </visual>
-      <inertial>
-        <origin rpy="0 0 0" xyz="0.000000 0.000000 0.000000"/>
-        <mass value="0.0001"/>
-        <inertia ixx="1e-08" ixy="0" ixz="0" iyy="1e-08" iyz="0" izz="1e-08"/>
-      </inertial>
-    </link>
-    <!-- Finger mesh index -->
-    <!--mesh filename="package://baxter_description/meshes/electric_gripper/fingers/00017816.DAE" /--> <!--basic_hard_tip-->
-    <!--mesh filename="package://baxter_description/meshes/electric_gripper/fingers/00030515.DAE" /--> <!--extended_wide -->
-    <!--mesh filename="package://baxter_description/meshes/electric_gripper/fingers/00030516.DAE" /--> <!-- standard_wide -->
-    <!--mesh filename="package://baxter_description/meshes/electric_gripper/fingers/00030517.DAE" /--> <!-- standard_narrow -->
-    <!--mesh filename="package://baxter_description/meshes/electric_gripper/fingers/00030518.DAE" /--> <!--extended_narrow /-->
-    <!--mesh filename="package://baxter_description/meshes/electric_gripper/fingers/00030535.DAE" /--> <!-- limiter -->
-    <!-- Right finger -->
-    <link name="${side}_gripper_r_finger">
-      <gravity>0</gravity>
-      <visual>
-        <origin rpy="0 1.57079632679 0" xyz="0.007 -0.036 0.0135"/>
-        <geometry>
-          <mesh filename="package://baxter_description/meshes/electric_gripper/fingers/extended_narrow.DAE" /> <!-- Long left finger-->
-        </geometry>
-      </visual>
-      <collision>
-        <origin rpy="0 1.57079632679 0" xyz="0.007 -0.036 0.0135"/>
-        <geometry>
-          <mesh filename="package://baxter_description/meshes/electric_gripper/fingers/extended_narrow.DAE" /> <!-- Long left finger-->
-        </geometry>
-      </collision>
-      <inertial>
-        <origin rpy="0 1.57079632679 0" xyz="0.007 -0.036 0.0135"/>
-        <!-- <mass value="0.00094542"/> -->
-        <!-- <inertia ixx="2e-08" ixy="0" ixz="0" iyy="3e-08" iyz="0" izz="2e-08"/> -->
-        <mass value="0.01"/>
-        <inertia ixx="0.01" ixy="0" ixz="0" iyy="0.01" iyz="0" izz="0.01"/>
-      </inertial>
-    </link>
+    <!-- Left finger link -->
+    <xacro:include filename="$(find baxter_description)/urdf/${l_finger}.xacro" />
+    <xacro:finger_xacro gripper_side="${side}" finger_side="l" reflect="1" finger_tip="${l_finger_tip}" add_finger_tip="${add_l_finger_tip}"/>
+    <!-- Right finger link -->
+    <xacro:include filename="$(find baxter_description)/urdf/${r_finger}.xacro" />
+    <xacro:finger_xacro gripper_side="${side}" finger_side="r" reflect="-1" finger_tip="${r_finger_tip}" add_finger_tip="${add_r_finger_tip}"/>
+    <!-- Electric Gripper Base -->
+    <joint name="${gripper_side}_gripper_electric_base_joint" type="fixed">
+      <origin rpy="0 0 0" xyz="0 0 0.025"/>
+      <parent link="${side}_gripper_base"/>
+      <child link="${side}_gripper_electric_base"/>
+    </joint>
     <!-- Left finger -->
-    <link name="${side}_gripper_l_finger">
-      <gravity>0</gravity>
-      <visual>
-        <origin rpy="0 -1.57079632679 0" xyz="0.007 -0.036 -0.0135"/>
-        <geometry>
-          <mesh filename="package://baxter_description/meshes/electric_gripper/fingers/extended_narrow.DAE" />
-        </geometry>
-      </visual>
-      <collision>
-        <origin rpy="0 -1.57079632679 0" xyz="0.007 -0.036 -0.0135"/>
-        <geometry>
-          <mesh filename="package://baxter_description/meshes/electric_gripper/fingers/extended_narrow.DAE" /> <!-- Long left finger-->
-        </geometry>
-      </collision>
-      <inertial>
-        <origin rpy="0 -1.57079632679 0" xyz="0.007 -0.036 -0.0135"/>
-        <!-- <mass value="0.00094542"/> -->
-        <!-- <inertia ixx="2e-08" ixy="0" ixz="0" iyy="3e-08" iyz="0" izz="2e-08"/> -->
-        <mass value="0.01"/>
-        <inertia ixx="0.01" ixy="0" ixz="0" iyy="0.01" iyz="0" izz="0.01"/>
-      </inertial>
-    </link>
-    <!-- Base of Right end effector -->
-    <joint name="${side}_endpoint" type="fixed">
-      <origin rpy="1.57      0 0" xyz="-0.005 0.0 0.02"/>
-      <parent link="${side}_hand"/>
-      <child link="${side}_gripper"/>
+    <joint name="${gripper_side}_gripper_l_finger_joint" type="prismatic">
+      <origin rpy="0 0 0" xyz="0.0 ${(l_finger_slot-1)*0.0095-0.011} 0.017"/>
+      <axis xyz="0 1 0"/>
+      <parent link="${side}_gripper_electric_base"/>
+      <child link="${side}_gripper_l_finger"/>
+      <limit effort="20.0" lower="${(l_finger_slot-1)*0.0095-0.011 + 0.020833}" upper="${(l_finger_slot-1)*0.0095-0.011}" velocity="5.0"/>
+      <dynamics damping="0.7" friction="0.0"/>
     </joint>
     <!-- Right finger -->
     <joint name="${gripper_side}_gripper_r_finger_joint" type="prismatic">
-      <origin rpy="0 0 0" xyz="0.0 0.06 -0.035"/>
-      <axis xyz="0 0 1"/>
-      <parent link="${side}_gripper"/>
+      <origin rpy="0 0 0" xyz="0.0 ${(r_finger_slot-1)*-0.0095+0.011} 0.017"/>
+      <axis xyz="0 1 0"/>
+      <parent link="${side}_gripper_electric_base"/>
       <child link="${side}_gripper_r_finger"/>
-      <limit effort="20.0" lower="-0.0095" upper="0.0215" velocity="5.0"/> <!-- upper is open -->
+      <limit effort="20.0" lower="${(r_finger_slot-1)*-0.0095+0.011 - 0.020833}" upper="${(r_finger_slot-1)*-0.0095+0.011}" velocity="5.0"/>
       <dynamics damping="0.7" friction="0.0"/>
-    </joint>
-    <!-- Left finger -->
-    <joint name="${gripper_side}_gripper_l_finger_joint" type="prismatic">
-      <origin rpy="0 0 0" xyz="0.0 0.06 0.035"/>
-      <axis xyz="0 0 1"/>
-      <parent link="${side}_gripper"/>
-      <child link="${side}_gripper_l_finger"/>
-      <limit effort="20.0" lower="-0.0215" upper="0.0095" velocity="5.0"/> <!-- mimic joint for lower is open -->
-      <dynamics damping="0.7" friction="0.0"/>
-      <mimic joint="${gripper_side}_gripper_r_finger_joint" offset="0"
-             multiplier="-1" />
     </joint>
     <transmission name="gripper_${side}1">
