Commit message: Moved urdf and meshes to rethink_ee_description pkg

File: baxter_description/urdf/left_end_effector.urdf.xacro (robot description, xacro)
@@ -1,5 +1,5 @@
 <?xml version="1.0" ?>
 <robot name="left_end_effector" xmlns:xacro="http://www.ros.org/wiki/xacro">
-  <xacro:include filename="$(find baxter_description)/urdf/electric_gripper/rethink_electric_gripper.xacro" />
+  <xacro:include filename="$(find rethink_ee_description)/urdf/electric_gripper/rethink_electric_gripper.xacro" />
   <xacro:rethink_electric_gripper side="left"
                                   l_finger="extended_narrow"

File: baxter_description/urdf/right_end_effector.urdf.xacro (robot description, xacro)
@@ -1,5 +1,5 @@
 <?xml version="1.0" ?>
 <robot name="right_end_effector" xmlns:xacro="http://www.ros.org/wiki/xacro">
-  <xacro:include filename="$(find baxter_description)/urdf/electric_gripper/rethink_electric_gripper.xacro" />
+  <xacro:include filename="$(find rethink_ee_description)/urdf/electric_gripper/rethink_electric_gripper.xacro" />
   <xacro:rethink_electric_gripper side="right"
                                   l_finger="standard_narrow"

File: rethink_ee_description/urdf/electric_gripper/example_end_effector.urdf.xacro (robot description, xacro)
@@ -1,5 +1,5 @@
 <?xml version="1.0"?>
 <robot xmlns:xacro="http://www.ros.org/wiki/xacro" name="left_electric_gripper">
-  <xacro:include filename="$(find baxter_description)/urdf/electric_gripper/rethink_electric_gripper.xacro" />
+  <xacro:include filename="$(find rethink_ee_description)/urdf/electric_gripper/rethink_electric_gripper.xacro" />
   <xacro:rethink_electric_gripper side="left"
                                   l_finger="extended_narrow"

File: rethink_ee_description/urdf/electric_gripper/fingers/basic_hard_tip.xacro (robot description, xacro)
@@ -1,4 +1,4 @@
 <?xml version="1.0"?>
-<robot xmlns:xacro="http://www.ros.org/wiki/xacro" name="basic_soft_tip">
+<robot xmlns:xacro="http://www.ros.org/wiki/xacro" name="basic_hard_tip">
   <xacro:macro name="finger_tip_xacro" params="parent_link reflect grasp *joint_origin">
     <xacro:property name="g_reflect" value="${reflect}" scope="local"/>
@@ -10,5 +10,5 @@
         <origin rpy="0 0 ${pi*(g_reflect+1)/2}" xyz="0 0 0"/>
         <geometry>
-          <mesh filename="package://baxter_description/meshes/electric_gripper/fingers/basic_soft_tip.DAE" />
+          <mesh filename="package://rethink_ee_description/meshes/electric_gripper/fingers/basic_hard_tip.DAE" />
         </geometry>
       </visual>
@@ -16,5 +16,5 @@
         <origin rpy="0 0 ${pi*(g_reflect+1)/2}" xyz="0 ${-0.0045*g_reflect} -0.015"/>
         <geometry>
-          <box size="0.016 0.007 0.037"/>
+          <box size="0.016 0.0065 0.037"/>
         </geometry>
       </collision>

File: rethink_ee_description/urdf/electric_gripper/fingers/basic_soft_tip.xacro (robot description, xacro)
@@ -1,4 +1,4 @@
 <?xml version="1.0"?>
-<robot xmlns:xacro="http://www.ros.org/wiki/xacro" name="half_round_tip">
+<robot xmlns:xacro="http://www.ros.org/wiki/xacro" name="basic_soft_tip">
   <xacro:macro name="finger_tip_xacro" params="parent_link reflect grasp *joint_origin">
     <xacro:property name="g_reflect" value="${reflect}" scope="local"/>
@@ -10,5 +10,5 @@
         <origin rpy="0 0 ${pi*(g_reflect+1)/2}" xyz="0 0 0"/>
         <geometry>
-          <mesh filename="package://baxter_description/meshes/electric_gripper/fingers/half_round_tip.DAE" />
+          <mesh filename="package://rethink_ee_description/meshes/electric_gripper/fingers/basic_soft_tip.DAE" />
         </geometry>
       </visual>
@@ -16,5 +16,5 @@
         <origin rpy="0 0 ${pi*(g_reflect+1)/2}" xyz="0 ${-0.0045*g_reflect} -0.015"/>
         <geometry>
-          <cylinder length="0.037" radius="0.008"/>
+          <box size="0.016 0.007 0.037"/>
         </geometry>
       </collision>

File: rethink_ee_description/urdf/electric_gripper/fingers/extended_narrow.xacro (robot description, xacro)
@@ -1,18 +1,18 @@
 <?xml version="1.0"?>
-<robot xmlns:xacro="http://www.ros.org/wiki/xacro" name="wide_extended">
+<robot xmlns:xacro="http://www.ros.org/wiki/xacro" name="extended_narrow">
   <xacro:macro name="finger_xacro" params="gripper_side finger_side reflect finger_tip finger_grasp">
-    <xacro:property name="finger_length" value="0.1127" scope="global"/>
-    <xacro:property name="finger_width" value="0.05503" scope="local"/>
+  <xacro:property name="finger_length" value="0.1127" scope="global"/>
+  <xacro:property name="finger_width" value="0.01725" scope="local"/>
     <link name="${gripper_side}_gripper_${finger_side}_finger">
       <visual>
         <origin rpy="0 0 ${-pi/2*(reflect+1)}" xyz="0 0 0"/>
         <geometry>
-          <mesh filename="package://baxter_description/meshes/electric_gripper/fingers/extended_wide.DAE" />
+          <mesh filename="package://rethink_ee_description/meshes/electric_gripper/fingers/extended_narrow.DAE" />
         </geometry>
       </visual>
-     <xacro:property name="finger_box_height" value="0.01" scope="local"/>
-     <xacro:property name="finger_box_width" value="0.0135" scope="local"/>
-     <xacro:property name="finger_box_length" value="0.0615" scope="local"/>
-     <collision>
+      <xacro:property name="finger_box_height" value="0.01" scope="local"/>
+      <xacro:property name="finger_box_width" value="0.0135" scope="local"/>
+      <xacro:property name="finger_box_length" value="0.0615" scope="local"/>
+      <collision>
         <origin rpy="0 0 ${-pi/2*(reflect+1)}" xyz="0 ${finger_width*reflect} ${finger_box_length}"/>
         <geometry>
@@ -24,5 +24,5 @@
       <xacro:property name="knuckle_box_length" value="${finger_width + 0.03275}" scope="local"/>
       <collision>
-        <origin rpy="0 0 ${-pi/2*(reflect+1)}" xyz="${reflect*-0.005} ${0.016*reflect} 0.0083"/>
+        <origin rpy="0 0 ${-pi/2*(reflect+1)}" xyz="${reflect*-0.005} ${-0.003*reflect} 0.0083"/>
         <geometry>
           <box size="${knuckle_box_height} ${knuckle_box_length} ${knuckle_box_width}"/>
@@ -46,5 +46,5 @@
      <xacro:property name="finger_tip" value="none" scope="local"/>
    </xacro:if>
-   <xacro:include filename="$(find baxter_description)/urdf/electric_gripper/fingers/${finger_tip}.xacro" />
+   <xacro:include filename="$(find rethink_ee_description)/urdf/electric_gripper/fingers/${finger_tip}.xacro" />
    <xacro:finger_tip_xacro parent_link="${gripper_side}_gripper_${finger_side}_finger" reflect="${reflect}" grasp="${finger_grasp}">
        <origin rpy="0 0 0" xyz="0.0 ${reflect*finger_width} ${finger_length}"/>

File: rethink_ee_description/urdf/electric_gripper/fingers/extended_wide.xacro (robot description, xacro)
@@ -1,18 +1,18 @@
 <?xml version="1.0"?>
-<robot xmlns:xacro="http://www.ros.org/wiki/xacro" name="extended_narrow">
+<robot xmlns:xacro="http://www.ros.org/wiki/xacro" name="wide_extended">
   <xacro:macro name="finger_xacro" params="gripper_side finger_side reflect finger_tip finger_grasp">
-  <xacro:property name="finger_length" value="0.1127" scope="global"/>
-  <xacro:property name="finger_width" value="0.01725" scope="local"/>
+    <xacro:property name="finger_length" value="0.1127" scope="global"/>
+    <xacro:property name="finger_width" value="0.05503" scope="local"/>
     <link name="${gripper_side}_gripper_${finger_side}_finger">
       <visual>
         <origin rpy="0 0 ${-pi/2*(reflect+1)}" xyz="0 0 0"/>
         <geometry>
-          <mesh filename="package://baxter_description/meshes/electric_gripper/fingers/extended_narrow.DAE" />
+          <mesh filename="package://rethink_ee_description/meshes/electric_gripper/fingers/extended_wide.DAE" />
         </geometry>
       </visual>
-      <xacro:property name="finger_box_height" value="0.01" scope="local"/>
-      <xacro:property name="finger_box_width" value="0.0135" scope="local"/>
-      <xacro:property name="finger_box_length" value="0.0615" scope="local"/>
-      <collision>
+     <xacro:property name="finger_box_height" value="0.01" scope="local"/>
+     <xacro:property name="finger_box_width" value="0.0135" scope="local"/>
+     <xacro:property name="finger_box_length" value="0.0615" scope="local"/>
+     <collision>
         <origin rpy="0 0 ${-pi/2*(reflect+1)}" xyz="0 ${finger_width*reflect} ${finger_box_length}"/>
         <geometry>
@@ -24,5 +24,5 @@
       <xacro:property name="knuckle_box_length" value="${finger_width + 0.03275}" scope="local"/>
       <collision>
-        <origin rpy="0 0 ${-pi/2*(reflect+1)}" xyz="${reflect*-0.005} ${-0.003*reflect} 0.0083"/>
+        <origin rpy="0 0 ${-pi/2*(reflect+1)}" xyz="${reflect*-0.005} ${0.016*reflect} 0.0083"/>
         <geometry>
           <box size="${knuckle_box_height} ${knuckle_box_length} ${knuckle_box_width}"/>
@@ -46,5 +46,5 @@
      <xacro:property name="finger_tip" value="none" scope="local"/>
    </xacro:if>
-   <xacro:include filename="$(find baxter_description)/urdf/electric_gripper/fingers/${finger_tip}.xacro" />
+   <xacro:include filename="$(find rethink_ee_description)/urdf/electric_gripper/fingers/${finger_tip}.xacro" />
    <xacro:finger_tip_xacro parent_link="${gripper_side}_gripper_${finger_side}_finger" reflect="${reflect}" grasp="${finger_grasp}">
        <origin rpy="0 0 0" xyz="0.0 ${reflect*finger_width} ${finger_length}"/>

File: rethink_ee_description/urdf/electric_gripper/fingers/half_round_tip.xacro (robot description, xacro)
@@ -1,4 +1,4 @@
 <?xml version="1.0"?>
-<robot xmlns:xacro="http://www.ros.org/wiki/xacro" name="basic_hard_tip">
+<robot xmlns:xacro="http://www.ros.org/wiki/xacro" name="half_round_tip">
   <xacro:macro name="finger_tip_xacro" params="parent_link reflect grasp *joint_origin">
     <xacro:property name="g_reflect" value="${reflect}" scope="local"/>
@@ -10,5 +10,5 @@
         <origin rpy="0 0 ${pi*(g_reflect+1)/2}" xyz="0 0 0"/>
         <geometry>
-          <mesh filename="package://baxter_description/meshes/electric_gripper/fingers/basic_hard_tip.DAE" />
+          <mesh filename="package://rethink_ee_description/meshes/electric_gripper/fingers/half_round_tip.DAE" />
         </geometry>
       </visual>
@@ -16,5 +16,5 @@
         <origin rpy="0 0 ${pi*(g_reflect+1)/2}" xyz="0 ${-0.0045*g_reflect} -0.015"/>
         <geometry>
-          <box size="0.016 0.0065 0.037"/>
+          <cylinder length="0.037" radius="0.008"/>
         </geometry>
       </collision>

File: rethink_ee_description/urdf/electric_gripper/fingers/paddle_tip.xacro (robot description, xacro)
@@ -10,5 +10,5 @@
         <origin rpy="0 0 ${pi*(g_reflect+1)/2}" xyz="0 0 0"/>
         <geometry>
-          <mesh filename="package://baxter_description/meshes/electric_gripper/fingers/paddle_tip.DAE" />
+          <mesh filename="package://rethink_ee_description/meshes/electric_gripper/fingers/paddle_tip.DAE" />
         </geometry>
       </visual>

File: rethink_ee_description/urdf/electric_gripper/fingers/standard_narrow.xacro (robot description, xacro)
@@ -8,5 +8,5 @@
         <origin rpy="0 0 ${-pi/2*(reflect+1)}" xyz="0 0 0"/>
         <geometry>
-          <mesh filename="package://baxter_description/meshes/electric_gripper/fingers/standard_narrow.DAE" />
+          <mesh filename="package://rethink_ee_description/meshes/electric_gripper/fingers/standard_narrow.DAE" />
         </geometry>
       </visual>
@@ -46,5 +46,5 @@
      <xacro:property name="finger_tip" value="none" scope="local"/>
    </xacro:if>
-   <xacro:include filename="$(find baxter_description)/urdf/electric_gripper/fingers/${finger_tip}.xacro" />
+   <xacro:include filename="$(find rethink_ee_description)/urdf/electric_gripper/fingers/${finger_tip}.xacro" />
    <xacro:finger_tip_xacro parent_link="${gripper_side}_gripper_${finger_side}_finger" reflect="${reflect}" grasp="${finger_grasp}">
        <origin rpy="0 0 0" xyz="0.0 ${reflect*finger_width} ${finger_length}"/>

File: rethink_ee_description/urdf/electric_gripper/fingers/standard_wide.xacro (robot description, xacro)
@@ -8,5 +8,5 @@
         <origin rpy="0 0 ${-pi/2*(reflect+1)}" xyz="0 0 0"/>
         <geometry>
-          <mesh filename="package://baxter_description/meshes/electric_gripper/fingers/standard_wide.DAE" />
+          <mesh filename="package://rethink_ee_description/meshes/electric_gripper/fingers/standard_wide.DAE" />
         </geometry>
       </visual>
@@ -46,5 +46,5 @@
      <xacro:property name="finger_tip" value="none" scope="local"/>
    </xacro:if>
-   <xacro:include filename="$(find baxter_description)/urdf/electric_gripper/fingers/${finger_tip}.xacro" />
+   <xacro:include filename="$(find rethink_ee_description)/urdf/electric_gripper/fingers/${finger_tip}.xacro" />
    <xacro:finger_tip_xacro parent_link="${gripper_side}_gripper_${finger_side}_finger" reflect="${reflect}" grasp="${finger_grasp}">
        <origin rpy="0 0 0" xyz="0.0 ${reflect*finger_width} ${finger_length}"/>

File: rethink_ee_description/urdf/electric_gripper/rethink_electric_gripper.xacro (robot description, xacro)
@@ -8,5 +8,5 @@
         <origin rpy="${-pi/2} ${pi} 0" xyz="0 0 0"/>
         <geometry>
-          <mesh filename="package://baxter_description/meshes/electric_gripper/electric_gripper_base.DAE"/>
+          <mesh filename="package://rethink_ee_description/meshes/electric_gripper/electric_gripper_base.DAE"/>
         </geometry>
       </visual>
@@ -28,9 +28,9 @@
     <!-- Left finger link -->
     <xacro:property name="finger_length" value="0.0" scope="global"/>
-    <xacro:include filename="$(find baxter_description)/urdf/electric_gripper/fingers/${l_finger}.xacro" />
+    <xacro:include filename="$(find rethink_ee_description)/urdf/electric_gripper/fingers/${l_finger}.xacro" />
     <xacro:finger_xacro gripper_side="${side}" finger_side="l" reflect="1" finger_tip="${l_finger_tip}" finger_grasp="${l_finger_grasp}"/>
     <xacro:property name="tip_finger_length" value="${finger_length}" scope="local"/>
     <!-- Right finger link -->
-    <xacro:include filename="$(find baxter_description)/urdf/electric_gripper/fingers/${r_finger}.xacro" />
+    <xacro:include filename="$(find rethink_ee_description)/urdf/electric_gripper/fingers/${r_finger}.xacro" />
     <xacro:finger_xacro gripper_side="${side}" finger_side="r" reflect="-1" finger_tip="${r_finger_tip}" finger_grasp="${r_finger_grasp}"/>
     <xacro:if value="${finger_length > tip_finger_length}">

File: rethink_ee_description/urdf/vacuum_gripper/custom_vacuum_gripper.xacro (robot description, xacro)
@@ -7,5 +7,5 @@
         <origin rpy="${-pi/2} ${pi} 0" xyz="0 0 0"/>
         <geometry>
-          <mesh filename="package://baxter_description/meshes/pneumatic_grippers_base.DAE"/>
+          <mesh filename="package://rethink_ee_description/meshes/pneumatic_grippers_base.DAE"/>
         </geometry>
       </visual>

File: rethink_ee_description/urdf/vacuum_gripper/example_end_effector.urdf.xacro (robot description, xacro)
@@ -1,5 +1,5 @@
 <?xml version="1.0"?>
 <robot xmlns:xacro="http://www.ros.org/wiki/xacro" name="left_electric_gripper">
-  <xacro:include filename="$(find baxter_description)/urdf/electric_gripper/rethink_electric_gripper.xacro" />
+  <xacro:include filename="$(find rethink_ee_description)/urdf/electric_gripper/rethink_electric_gripper.xacro" />
   <xacro:rethink_electric_gripper side="left"
                                   gripper_side="l"

File: rethink_ee_description/urdf/vacuum_gripper/rethink_vacuum_gripper.xacro (robot description, xacro)
@@ -7,5 +7,5 @@
         <origin rpy="${-pi/2} ${pi} 0" xyz="0 0 0"/>
         <geometry>
-          <mesh filename="package://baxter_description/meshes/pneumatic_grippers_w_cup.DAE"/>
+          <mesh filename="package://rethink_ee_description/meshes/pneumatic_grippers_w_cup.DAE"/>
         </geometry>
       </visual>
