Commit message: Adds Support for External EndEffector modification
- Reverted baxter.urdf to original for backward compatibility
- Created baxter.urdf.xacro as the default URDF
- End effectors are now required, even if just using null grippers
- <side>_endpoint joint and <side>_gripper end effector link is now
  used to be consistent with the robot and take advantage of onboard IK
- Finally fixed the pneumatic gripper to work just line the electric
  gripper in terms of xacro URDF construction
- Renamed vacuum gripper back to pneumatic gripper to be constent with
  onboard robot

File: baxter_description/urdf/baxter.urdf.xacro (robot description, xacro)
@@ -3,18 +3,15 @@
   <!-- Arguments and Defaults-->
   <xacro:arg name="gazebo" default="false"/>
-  <xacro:arg name="left_end_effector" default="true"/>
-  <xacro:arg name="right_end_effector" default="true"/>
   <!-- Baxter Base URDF -->
-  <xacro:include filename="$(find baxter_description)/urdf/baxter.urdf" />
+  <xacro:include filename="$(find baxter_description)/urdf/baxter_base/baxter_base.xacro" />
+  <!-- Gazebo Tags -->
   <xacro:if value="$(arg gazebo)">
       <xacro:include filename="$(find baxter_description)/urdf/gazebo/baxter.gazebo.xacro" />
   </xacro:if>
+  <!-- Baxter Pedestal -->
+  <xacro:include filename="$(find baxter_description)/urdf/pedestal/pedestal.xacro" />
   <!-- Left End Effector -->
-  <xacro:if value="$(arg left_end_effector)">
-    <xacro:include filename="$(find baxter_description)/urdf/left_end_effector.urdf.xacro" />
-  </xacro:if>
+  <xacro:include filename="$(find baxter_description)/urdf/left_end_effector.urdf.xacro" />
   <!-- Right End Effector -->
-  <xacro:if value="$(arg right_end_effector)">
-    <xacro:include filename="$(find baxter_description)/urdf/right_end_effector.urdf.xacro" />
-  </xacro:if>
+  <xacro:include filename="$(find baxter_description)/urdf/right_end_effector.urdf.xacro" />
 </robot>

File: baxter_description/urdf/baxter_base/baxter_base.xacro (robot description, xacro)
@@ -1,10 +1,3 @@
 <?xml version="1.0" ?>
-<!-- ============================================================================================== -->
-<!-- |                                                                                            | -->
-<!-- |    baxter.urdf is DEPRECATED. It is included here for backward compatibility.              | -->
-<!-- |    Please use baxter.urdf.xacro by running:                                                | -->
-<!-- |$ rosrun xacro xacro.py - -inorder `rospack find baxter_description`/urdf/baxter.urdf.xacro | -->
-<!-- |                                                                                            | -->
-<!-- ============================================================================================== -->
 <robot name="baxter">
   <link name="base">
@@ -16,4 +9,7 @@
         <mesh filename="package://baxter_description/meshes/torso/base_link.DAE"/>
       </geometry>
+      <material name="darkgray">
+        <color rgba=".2 .2 .2 1"/>
+      </material>
     </visual>
     <collision>
@@ -41,26 +37,4 @@
       <mass value="0.0001"/>
       <inertia ixx="1e-08" ixy="0" ixz="0" iyy="1e-08" iyz="0" izz="1e-08"/>
-    </inertial>
-  </link>
-  <link name="pedestal">
-    <visual>
-      <origin rpy="0 0 0" xyz="0 0 0"/>
-      <geometry>
-        <mesh filename="package://baxter_description/meshes/base/PEDESTAL.DAE"/>
-      </geometry>
-      <material name="darkgray">
-        <color rgba=".2 .2 .2 1"/>
-      </material>
-    </visual>
-    <collision>
-      <origin rpy="0 0 0" xyz="0 0 0"/>
-      <geometry>
-        <mesh filename="package://baxter_description/meshes/base/pedestal_link_collision.DAE"/>
-      </geometry>
-    </collision>
-    <inertial>
-      <origin rpy="0 0 0" xyz="0 0 0"/>
-      <mass value="60.86397744"/>
-      <inertia ixx="5.0635929" ixy="0.00103417" ixz="0.80199628" iyy="6.08689388" iyz="0.00105311" izz="4.96191932"/>
     </inertial>
   </link>
@@ -236,9 +210,4 @@
     <child link="right_torso_itb"/>
   </joint>
-  <joint name="pedestal_fixed" type="fixed">
-    <origin rpy="0 0 0" xyz="0.0 0.0 0.0"/>
-    <parent link="torso"/>
-    <child link="pedestal"/>
-  </joint>
   <joint name="head_pan" type="revolute">
     <origin rpy="0 0 0" xyz="0.06 0 0.686"/>
@@ -246,5 +215,5 @@
     <parent link="torso"/>
     <child link="head"/>
-    <limit effort="50000" lower="-1.57079632679" upper="1.57079632679" velocity="10000"/>
+    <limit effort="50000" lower="-1.3963" upper="1.3963" velocity="10000"/>
     <dynamics damping="0.7" friction="0.0"/>
   </joint>
@@ -272,5 +241,4 @@
   <link name="right_arm_mount">
     <!-- all defaults -->
- <gravity>0</gravity>
     <inertial>
       <origin rpy="0 0 0" xyz="0 0 0"/>
@@ -280,5 +248,4 @@
   </link>
   <link name="right_upper_shoulder">
- <gravity>0</gravity>
     <visual>
       <origin rpy="0 0 0" xyz="0 0 0"/>
@@ -303,5 +270,4 @@
   </link>
   <link name="right_lower_shoulder">
- <gravity>0</gravity>
     <visual>
       <origin rpy="0 0 0" xyz="0 0 0"/>
@@ -326,5 +292,4 @@
   </link>
   <link name="right_upper_elbow">
- <gravity>0</gravity>
     <visual>
       <origin rpy="0 0 0" xyz="0 0 0"/>
@@ -349,5 +314,4 @@
   </link>
   <link name="right_upper_elbow_visual">
- <gravity>0</gravity>
     <collision>
       <origin rpy="0 0 0" xyz="0 0 0.1365"/>
@@ -363,5 +327,4 @@
   </link>
   <link name="right_lower_elbow">
- <gravity>0</gravity>
     <visual>
       <origin rpy="0 0 0" xyz="0 0 0"/>
@@ -386,5 +349,4 @@
   </link>
   <link name="right_upper_forearm">
- <gravity>0</gravity>
     <visual>
       <origin rpy="0 0 0" xyz="0 0 0"/>
@@ -409,5 +371,4 @@
   </link>
   <link name="right_upper_forearm_visual">
- <gravity>0</gravity>
     <collision>
       <origin rpy="0 0 0" xyz="0 0 0.136"/>
@@ -423,5 +384,4 @@
   </link>
   <link name="right_arm_itb">
- <gravity>0</gravity>
     <inertial>
       <origin rpy="0 0 0" xyz="0.000000 0.000000 0.000000"/>
@@ -431,5 +391,4 @@
   </link>
   <link name="right_lower_forearm">
- <gravity>0</gravity>
     <visual>
       <origin rpy="0 0 0" xyz="0 0 0"/>
@@ -454,5 +413,4 @@
   </link>
   <link name="right_wrist">
- <gravity>0</gravity>
     <visual>
       <origin rpy="0 0 0" xyz="0 0 0"/>
@@ -477,5 +435,4 @@
   </link>
   <link name="right_hand">
- <gravity>0</gravity>
     <collision>
       <origin rpy="0 0 0" xyz="0 0 -0.0232"/>
@@ -491,5 +448,4 @@
   </link>
   <link name="right_hand_camera">
- <gravity>0</gravity>
     <visual>
       <origin rpy="0 0 0" xyz="0 0 0"/>
@@ -508,5 +464,4 @@
   </link>
   <link name="right_hand_camera_axis">
- <gravity>0</gravity>
     <inertial>
       <origin rpy="0 0 0" xyz="0 0 0"/>
@@ -516,5 +471,4 @@
   </link>
   <link name="right_hand_range">
- <gravity>0</gravity>
     <visual>
       <origin rpy="0 0 0" xyz="0 0 0"/>
@@ -533,39 +487,4 @@
   </link>
   <link name="right_hand_accelerometer">
- <gravity>0</gravity>
-    <visual>
-      <origin rpy="0 0 0" xyz="0 0 0"/>
-      <geometry>
-        <box size="0.01 0.01 0.01"/>
-      </geometry>
-      <material name="black">
-        <color rgba="0 0 0 1"/>
-      </material>
-    </visual>
-    <inertial>
-      <origin rpy="0 0 0" xyz="0.000000 0.000000 0.000000"/>
-      <mass value="0.0001"/>
-      <inertia ixx="1e-08" ixy="0" ixz="0" iyy="1e-08" iyz="0" izz="1e-08"/>
-    </inertial>
-  </link>
-  <link name="right_gripper_base">
- <gravity>0</gravity>
-    <visual>
-      <origin rpy="0 0 0" xyz="0 0 -0.02"/>
-      <geometry>
-        <box size="0.025 0.075 0.035"/>
-      </geometry>
-      <material name="darkred">
-        <color rgba=".5 .1 .1 1"/>
-      </material>
-    </visual>
-    <inertial>
-      <origin rpy="0 0 0" xyz="0.000000 0.000000 0.000000"/>
-      <mass value="0.0001"/>
-      <inertia ixx="1e-08" ixy="0" ixz="0" iyy="1e-08" iyz="0" izz="1e-08"/>
-    </inertial>
-  </link>
-  <link name="right_gripper">
- <gravity>0</gravity>
     <visual>
       <origin rpy="0 0 0" xyz="0 0 0"/>
@@ -601,5 +520,5 @@
     <parent link="right_upper_shoulder"/>
     <child link="right_lower_shoulder"/>
-    <limit effort="100.0" lower="-2.147" upper="1.047" velocity="1.5"/>
+    <limit effort="50.0" lower="-2.147" upper="1.047" velocity="1.5"/>
     <dynamics damping="0.7" friction="0.0"/>
   </joint>
@@ -667,5 +586,4 @@
     <parent link="right_wrist"/>
     <child link="right_hand"/>
-    <dynamics damping="0.7" friction="0.0"/>
   </joint>
   <joint name="right_hand_camera" type="fixed">
@@ -689,17 +607,6 @@
     <child link="right_hand_accelerometer"/>
   </joint>
-  <joint name="right_gripper_base" type="fixed">
-    <origin rpy="0 0 0" xyz="0 0 0"/>
-    <parent link="right_hand"/>
-    <child link="right_gripper_base"/>
-  </joint>
-  <joint name="right_endpoint" type="fixed">
-    <origin rpy="0 0 0" xyz="0.0 0 0.025"/>
-    <parent link="right_gripper_base"/>
-    <child link="right_gripper"/>
-  </joint>
   <link name="left_arm_mount">
     <!-- all defaults -->
- <gravity>0</gravity>
     <inertial>
       <origin rpy="0 0 0" xyz="0 0 0"/>
@@ -709,5 +616,4 @@
   </link>
   <link name="left_upper_shoulder">
- <gravity>0</gravity>
     <visual>
       <origin rpy="0 0 0" xyz="0 0 0"/>
@@ -732,5 +638,4 @@
   </link>
   <link name="left_lower_shoulder">
- <gravity>0</gravity>
     <visual>
       <origin rpy="0 0 0" xyz="0 0 0"/>
@@ -755,5 +660,4 @@
   </link>
   <link name="left_upper_elbow">
- <gravity>0</gravity>
     <visual>
       <origin rpy="0 0 0" xyz="0 0 0"/>
@@ -778,5 +682,4 @@
   </link>
   <link name="left_upper_elbow_visual">
- <gravity>0</gravity>
     <collision>
       <origin rpy="0 0 0" xyz="0 0 0.1365"/>
@@ -792,5 +695,4 @@
   </link>
   <link name="left_lower_elbow">
- <gravity>0</gravity>
     <visual>
       <origin rpy="0 0 0" xyz="0 0 0"/>
@@ -815,5 +717,4 @@
   </link>
   <link name="left_upper_forearm">
- <gravity>0</gravity>
     <visual>
       <origin rpy="0 0 0" xyz="0 0 0"/>
@@ -838,5 +739,4 @@
   </link>
   <link name="left_upper_forearm_visual">
- <gravity>0</gravity>
     <collision>
       <origin rpy="0 0 0" xyz="0 0 0.136"/>
@@ -852,5 +752,4 @@
   </link>
   <link name="left_arm_itb">
- <gravity>0</gravity>
     <inertial>
       <origin rpy="0 0 0" xyz="0.000000 0.000000 0.000000"/>
@@ -860,5 +759,4 @@
   </link>
   <link name="left_lower_forearm">
- <gravity>0</gravity>
     <visual>
       <origin rpy="0 0 0" xyz="0 0 0"/>
@@ -883,5 +781,4 @@
   </link>
   <link name="left_wrist">
- <gravity>0</gravity>
     <visual>
       <origin rpy="0 0 0" xyz="0 0 0"/>
@@ -906,5 +803,4 @@
   </link>
   <link name="left_hand">
- <gravity>0</gravity>
     <collision>
       <origin rpy="0 0 0" xyz="0 0 -0.0232"/>
@@ -920,5 +816,4 @@
   </link>
   <link name="left_hand_camera">
- <gravity>0</gravity>
     <visual>
       <origin rpy="0 0 0" xyz="0 0 0"/>
@@ -937,5 +832,4 @@
   </link>
   <link name="left_hand_camera_axis">
- <gravity>0</gravity>
     <inertial>
       <origin rpy="0 0 0" xyz="0 0 0"/>
@@ -945,5 +839,4 @@
   </link>
   <link name="left_hand_range">
- <gravity>0</gravity>
     <visual>
       <origin rpy="0 0 0" xyz="0 0 0"/>
@@ -962,39 +855,4 @@
   </link>
   <link name="left_hand_accelerometer">
- <gravity>0</gravity>
-    <visual>
-      <origin rpy="0 0 0" xyz="0 0 0"/>
-      <geometry>
-        <box size="0.01 0.01 0.01"/>
-      </geometry>
-      <material name="black">
-        <color rgba="0 0 0 1"/>
-      </material>
-    </visual>
-    <inertial>
-      <origin rpy="0 0 0" xyz="0.000000 0.000000 0.000000"/>
-      <mass value="0.0001"/>
-      <inertia ixx="1e-08" ixy="0" ixz="0" iyy="1e-08" iyz="0" izz="1e-08"/>
-    </inertial>
-  </link>
-  <link name="left_gripper_base">
- <gravity>0</gravity>
-    <visual>
-      <origin rpy="0 0 0" xyz="0 0 -0.02"/>
-      <geometry>
-        <box size="0.025 0.075 0.035"/>
-      </geometry>
-      <material name="darkred">
-        <color rgba=".5 .1 .1 1"/>
-      </material>
-    </visual>
-    <inertial>
-      <origin rpy="0 0 0" xyz="0.000000 0.000000 0.000000"/>
-      <mass value="0.0001"/>
-      <inertia ixx="1e-08" ixy="0" ixz="0" iyy="1e-08" iyz="0" izz="1e-08"/>
-    </inertial>
-  </link>
-  <link name="left_gripper">
- <gravity>0</gravity>
     <visual>
       <origin rpy="0 0 0" xyz="0 0 0"/>
@@ -1030,5 +888,5 @@
     <parent link="left_upper_shoulder"/>
     <child link="left_lower_shoulder"/>
-    <limit effort="100.0" lower="-2.147" upper="1.047" velocity="1.5"/>
+    <limit effort="50.0" lower="-2.147" upper="1.047" velocity="1.5"/>
     <dynamics damping="0.7" friction="0.0"/>
   </joint>
@@ -1096,5 +954,4 @@
     <parent link="left_wrist"/>
     <child link="left_hand"/>
-    <dynamics damping="0.7" friction="0.0"/>
   </joint>
   <joint name="left_hand_camera" type="fixed">
@@ -1118,435 +975,3 @@
     <child link="left_hand_accelerometer"/>
   </joint>
-  <joint name="left_gripper_base" type="fixed">
-    <origin rpy="0 0 0" xyz="0 0 0"/>
-    <parent link="left_hand"/>
-    <child link="left_gripper_base"/>
-  </joint>
-  <joint name="left_endpoint" type="fixed">
-    <origin rpy="0 0 0" xyz="0.0 0 0.025"/>
-    <parent link="left_gripper_base"/>
-    <child link="left_gripper"/>
-  </joint>
-  <!-- Transmissions -->
-  <!-- Right Arm -->
-  <transmission name="right_tran1">
-    <type>transmission_interface/SimpleTransmission</type>
-    <joint name="right_s0">
-      <hardwareInterface>EffortJointInterface</hardwareInterface>
-    </joint>
-    <actuator name="right_motor1">
-      <hardwareInterface>EffortJointInterface</hardwareInterface>
-      <mechanicalReduction>1</mechanicalReduction>
-    </actuator>
-  </transmission>
-  <transmission name="right_tran2">
-    <type>transmission_interface/SimpleTransmission</type>
-    <joint name="right_s1">
-      <hardwareInterface>EffortJointInterface</hardwareInterface>
-    </joint>
-    <actuator name="right_motor2">
-      <hardwareInterface>EffortJointInterface</hardwareInterface>
-      <mechanicalReduction>1</mechanicalReduction>
-    </actuator>
-  </transmission>
-  <transmission name="right_tran3">
-    <type>transmission_interface/SimpleTransmission</type>
-    <joint name="right_e0">
-      <hardwareInterface>EffortJointInterface</hardwareInterface>
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
File: baxter_description/urdf/right_end_effector.urdf.xacro (robot description, xacro)
@@ -1,13 +1,5 @@
 <?xml version="1.0" ?>
 <robot name="right_end_effector" xmlns:xacro="http://www.ros.org/wiki/xacro">
-  <xacro:include filename="$(find rethink_ee_description)/urdf/electric_gripper/rethink_electric_gripper.xacro" />
-  <xacro:rethink_electric_gripper side="right"
-                                  l_finger="standard_narrow"
-                                  l_finger_slot="2"
-                                  l_finger_tip="half_round_tip"
-                                  l_finger_grasp="inner"
-                                  r_finger="standard_narrow"
-                                  r_finger_slot="2"
-                                  r_finger_tip="half_round_tip"
-                                  r_finger_grasp="inner"/>
+  <xacro:include filename="$(find rethink_ee_description)/urdf/null_gripper/null_gripper.xacro" />
+  <xacro:null_gripper side="right"/>
 </robot>

File: rethink_ee_description/urdf/electric_gripper/rethink_electric_gripper.xacro (robot description, xacro)
@@ -4,5 +4,5 @@
     <xacro:property name="gripper_side" value="${side[0]}" scope="local"/>
     <!-- Base of end effector -->
-    <link name="${side}_gripper_electric_base">
+    <link name="${side}_gripper_base">
       <visual>
         <origin rpy="${-pi/2} ${pi} 0" xyz="0 0 0"/>
@@ -29,14 +29,26 @@
     <xacro:property name="finger_length" value="0.0" scope="global"/>
     <xacro:include filename="$(find rethink_ee_description)/urdf/electric_gripper/fingers/${l_finger}.xacro" />
-    <xacro:finger_xacro gripper_side="${side}" finger_side="l" reflect="1" finger_tip="${l_finger_tip}" finger_grasp="${l_finger_grasp}"/>
+    <xacro:finger_xacro gripper_side="${gripper_side}" finger_side="l" reflect="1" finger_tip="${l_finger_tip}" finger_grasp="${l_finger_grasp}"/>
     <xacro:property name="tip_finger_length" value="${finger_length}" scope="local"/>
     <!-- Right finger link -->
     <xacro:include filename="$(find rethink_ee_description)/urdf/electric_gripper/fingers/${r_finger}.xacro" />
-    <xacro:finger_xacro gripper_side="${side}" finger_side="r" reflect="-1" finger_tip="${r_finger_tip}" finger_grasp="${r_finger_grasp}"/>
+    <xacro:finger_xacro gripper_side="${gripper_side}" finger_side="r" reflect="-1" finger_tip="${r_finger_tip}" finger_grasp="${r_finger_grasp}"/>
     <xacro:if value="${finger_length > tip_finger_length}">
         <xacro:property name="tip_finger_length" value="${finger_length}" scope="local"/>
     </xacro:if>
-    <!-- Electric Gripper Convenience Tip link -->
-    <link name="${side}_gripper_tip">
+    <!-- Electric Gripper Base Joint -->
+    <joint name="${side}_gripper_base" type="fixed">
+      <origin rpy="0 0 0" xyz="0 0 0.025"/>
+      <parent link="${side}_hand"/>
+      <child link="${side}_gripper_base"/>
+    </joint>
+    <!-- Electric Gripper Tip joint -->
+    <joint name="${side}_endpoint" type="fixed">
+      <origin rpy="0 0 0" xyz="0 0 ${tip_finger_length+0.02}"/>
+      <parent link="${side}_gripper_base"/>
+      <child link="${side}_gripper"/>
+    </joint>
+    <!-- Electric Gripper Tip link -->
+    <link name="${side}_gripper">
       <inertial>
         <origin rpy="0 0 0" xyz="0 0 0"/>
@@ -45,10 +57,4 @@
       </inertial>
     </link>
-    <!-- Electric Gripper Base -->
-    <joint name="${gripper_side}_gripper_electric_base_joint" type="fixed">
-      <origin rpy="0 0 0" xyz="0 0 0.025"/>
-      <parent link="${side}_gripper_base"/>
-      <child link="${side}_gripper_electric_base"/>
-    </joint>
     <!-- Left finger -->
     <xacro:property name="l_finger_offset" value="${((l_finger_slot-1)*0.0095) -0.011}" scope="local"/>
@@ -56,6 +62,6 @@
       <origin rpy="0 0 0" xyz="0.0 ${l_finger_offset} 0.02"/>
       <axis xyz="0 1 0"/>
-      <parent link="${side}_gripper_electric_base"/>
-      <child link="${side}_gripper_l_finger"/>
+      <parent link="${side}_gripper_base"/>
+      <child link="${gripper_side}_gripper_l_finger"/>
       <limit effort="20.0" lower="0.0" upper="0.020833" velocity="5.0"/>
       <dynamics damping="0.7" friction="0.0"/>
@@ -66,15 +72,9 @@
       <origin rpy="0 0 0" xyz="0.0 ${r_finger_offset} 0.02"/>
       <axis xyz="0 1 0"/>
-      <parent link="${side}_gripper_electric_base"/>
-      <child link="${side}_gripper_r_finger"/>
+      <parent link="${side}_gripper_base"/>
+      <child link="${gripper_side}_gripper_r_finger"/>
       <limit effort="20.0" lower="-0.020833" upper="0.0" velocity="5.0"/>
       <mimic joint="${gripper_side}_gripper_l_finger_joint" multiplier="-1.0"/>
       <dynamics damping="0.7" friction="0.0"/>
-    </joint>
-    <!-- Electric Gripper Convenience Tip joint -->
-    <joint name="${gripper_side}_gripper_tip_joint" type="fixed">
-      <origin rpy="0 0 0" xyz="0 0.0 ${tip_finger_length+0.02}"/>
-      <parent link="${side}_gripper_electric_base"/>
-      <child link="${side}_gripper_tip"/>
     </joint>
     <transmission name="gripper_${side}1">

Commit message: Re #73 Fix Baxter's base link to world
This commit adds a Fixed dummy link to Gazebo
which locks down Baxter, preventing him from
wandering over time with respect to Gazebo world.

I added this to the pedestal xacro to allow
for the future possibility of a mobile Baxter URDF
that would not need this fixed link (or pedistal).

Additionally, I consolidated the gazebo tags into
the baxter_base folder and removed the unused top
level gazebo xacro for baxter.

File: baxter_description/urdf/baxter.urdf.xacro (robot description, xacro)
@@ -1,14 +1,13 @@
 <?xml version="1.0" ?>
 <robot name="baxter" xmlns:xacro="http://www.ros.org/wiki/xacro">
-  <!-- Arguments and Defaults-->
   <xacro:arg name="gazebo" default="false"/>
   <!-- Baxter Base URDF -->
-  <xacro:include filename="$(find baxter_description)/urdf/baxter_base/baxter_base.xacro" />
-  <!-- Gazebo Tags -->
-  <xacro:if value="$(arg gazebo)">
-      <xacro:include filename="$(find baxter_description)/urdf/gazebo/baxter.gazebo.xacro" />
-  </xacro:if>
+  <xacro:include filename="$(find baxter_description)/urdf/baxter_base/baxter_base.xacro">
+    <xacro:arg name="gazebo" value="${gazebo}"/>
+  </xacro:include>
   <!-- Baxter Pedestal -->
-  <xacro:include filename="$(find baxter_description)/urdf/pedestal/pedestal.xacro" />
+  <xacro:include filename="$(find baxter_description)/urdf/pedestal/pedestal.xacro">
+    <xacro:arg name="gazebo" value="${gazebo}"/>
+  </xacro:include>
   <!-- Left End Effector -->
   <xacro:include filename="$(find baxter_description)/urdf/left_end_effector.urdf.xacro" />

File: baxter_description/urdf/baxter_base/baxter_base.xacro (robot description, xacro)
@@ -1,4 +1,9 @@
 <?xml version="1.0" ?>
-<robot name="baxter">
+<robot name="baxter" xmlns:xacro="http://www.ros.org/wiki/xacro">
+  <xacro:arg name="gazebo" default="false"/>
+  <xacro:if value="$(arg gazebo)">
+    <!-- Gazebo Tags -->
+    <xacro:include filename="$(find baxter_description)/urdf/baxter_base/baxter_base.gazebo.xacro" />
+  </xacro:if>
   <link name="base">
   </link>

File: baxter_description/urdf/pedestal/pedestal.xacro (robot description, xacro)
@@ -1,4 +1,6 @@
 <?xml version="1.0" ?>
 <robot name="pedistal" xmlns:xacro="http://www.ros.org/wiki/xacro">
+  <!-- Arguments and Defaults-->
+  <xacro:arg name="gazebo" default="false"/>
   <link name="pedestal">
     <visual>
@@ -28,3 +30,11 @@
     <child link="pedestal"/>
   </joint>
+  <xacro:if value="$(arg gazebo)">
+    <!-- When using the pedistal, fix Baxter to Gazebo world with 'base' frame -->
+    <link name="world"/>
+    <joint name="fixed" type="fixed">
+      <parent link="world"/>
+      <child link="base"/>
+    </joint>
+  </xacro:if>
 </robot>
