Commit message: args work in progress

File: baxter_description/urdf/baxter.urdf.xacro (robot description, xacro)
@@ -11,6 +11,50 @@
   </xacro:include>
   <!-- Left End Effector -->
-  <xacro:include filename="$(find baxter_description)/urdf/left_end_effector.urdf.xacro" />
+  <!-- Gripper types: electric_gripper, pneumatic_gripper, null_gripper -->
+  <xacro:arg name="left_end_effector"         default="electric_gripper"/>
+  <!-- Thes args are only used if left_gripper is electric_gripper -->
+  <xacro:arg name="l_gripper_l_finger"        default="extended_narrow"/>
+  <xacro:arg name="l_gripper_l_finger_slot"   default="2"/>
+  <xacro:arg name="l_gripper_l_finger_tip"    default="paddle_tip"/>
+  <xacro:arg name="l_gripper_l_finger_grasp"  default="inner"/>
+  <xacro:arg name="l_gripper_r_finger"        default="standard_wide"/>
+  <xacro:arg name="l_gripper_r_finger_slot"   default="2"/>
+  <xacro:arg name="l_gripper_r_finger_tip"    default="paddle_tip"/>
+  <xacro:arg name="l_gripper_r_finger_grasp"  default="inner"/>
+  <xacro:include filename="$(find baxter_description)/urdf/left_end_effector.urdf.xacro">
+    <xacro:arg name="end_effector_type" value="$(arg left_end_effector)"/>
+    <xacro:arg name="l_finger"          value="$(arg l_gripper_l_finger)"/>
+    <xacro:arg name="l_finger_slot"     value="$(arg l_gripper_l_finger_slot)"/>
+    <xacro:arg name="l_finger_tip"      value="$(arg l_gripper_l_finger_tip)"/>
+    <xacro:arg name="l_finger_grasp"    value="$(arg l_gripper_l_finger_grasp)"/>
+    <xacro:arg name="l_finger_grasp"    value="$(arg l_gripper_r_finger)"/>
+    <xacro:arg name="r_finger_slot"     value="$(arg l_gripper_r_finger_slot)"/>
+    <xacro:arg name="r_finger_tip"      value="$(arg l_gripper_r_finger_tip)"/>
+    <xacro:arg name="r_finger_grasp"    value="$(arg l_gripper_r_finger_grasp)"/>
+    <xacro:arg name="gazebo"            value="$(arg gazebo)"/>
+  </xacro:include>
   <!-- Right End Effector -->
-  <xacro:include filename="$(find baxter_description)/urdf/right_end_effector.urdf.xacro" />
+  <!-- Gripper types: electric_gripper, pneumatic_gripper, null_gripper -->
+  <xacro:arg name="right_end_effector" default="electric_gripper"/>
+  <!-- Thes args are only used if right_gripper is electric_gripper -->
+  <xacro:arg name="r_gripper_l_finger"        default="extended_narrow"/>
+  <xacro:arg name="r_gripper_l_finger_slot"   default="2"/>
+  <xacro:arg name="r_gripper_l_finger_tip"    default="half_round_tip"/>
+  <xacro:arg name="r_gripper_l_finger_grasp"  default="inner"/>
+  <xacro:arg name="r_gripper_r_finger"        default="extended_narrow"/>
+  <xacro:arg name="r_gripper_r_finger_slot"   default="2"/>
+  <xacro:arg name="r_gripper_r_finger_tip"    default="half_round_tip"/>
+  <xacro:arg name="r_gripper_r_finger_grasp"  default="inner"/>
+  <xacro:include filename="$(find baxter_description)/urdf/right_end_effector.urdf.xacro">
+    <xacro:arg name="end_effector_type" value="$(arg right_end_effector)"/>
+    <xacro:arg name="l_finger"          value="$(arg r_gripper_l_finger)"/>
+    <xacro:arg name="l_finger_slot"     value="$(arg r_gripper_l_finger_slot)"/>
+    <xacro:arg name="l_finger_tip"      value="$(arg r_gripper_l_finger_tip)"/>
+    <xacro:arg name="l_finger_grasp"    value="$(arg r_gripper_l_finger_grasp)"/>
+    <xacro:arg name="l_finger_grasp"    value="$(arg r_gripper_r_finger)"/>
+    <xacro:arg name="r_finger_slot"     value="$(arg r_gripper_r_finger_slot)"/>
+    <xacro:arg name="r_finger_tip"      value="$(arg r_gripper_r_finger_tip)"/>
+    <xacro:arg name="r_finger_grasp"    value="$(arg r_gripper_r_finger_grasp)"/>
+    <xacro:arg name="gazebo"            value="$(arg gazebo)"/>
+  </xacro:include>
 </robot>

File: baxter_description/urdf/left_end_effector.urdf.xacro (robot description, xacro)
@@ -1,13 +1,37 @@
 <?xml version="1.0" ?>
 <robot name="left_end_effector" xmlns:xacro="http://www.ros.org/wiki/xacro">
-  <xacro:include filename="$(find rethink_ee_description)/urdf/electric_gripper/rethink_electric_gripper.xacro" />
-  <xacro:rethink_electric_gripper side="left"
-                                  l_finger="extended_narrow"
-                                  l_finger_slot="2"
-                                  l_finger_tip="paddle_tip"
-                                  l_finger_grasp="inner"
-                                  r_finger="extended_narrow"
-                                  r_finger_slot="2"
-                                  r_finger_tip="paddle_tip"
-                                  r_finger_grasp="inner"/>
+  <xacro:property name="side" value="left" scope="local"/>
+  <xacro:arg name="end_effector_type" default="electric_gripper" scope="local"/>
+  <xacro:arg name="gazebo"            default="false" scope="local"/>
+  <xacro:if value="${'$(arg end_effector_type)' == 'electric_gripper'}">
+    <!-- Left Electric Gripper -->
+    <xacro:arg name="l_finger"        default="extended_narrow" scope="local"/>
+    <xacro:arg name="l_finger_slot"   default="2" scope="local"/>
+    <xacro:arg name="l_finger_tip"    default="paddle_tip" scope="local"/>
+    <xacro:arg name="l_finger_grasp"  default="inner" scope="local"/>
+    <xacro:arg name="r_finger"        default="standard_wide" scope="local"/>
+    <xacro:arg name="r_finger_slot"   default="2" scope="local"/>
+    <xacro:arg name="r_finger_tip"    default="paddle_tip" scope="local"/>
+    <xacro:arg name="r_finger_grasp"  default="inner" scope="local"/>
+    <xacro:include filename="$(find rethink_ee_description)/urdf/electric_gripper/rethink_electric_gripper.xacro"/>
+    <xacro:rethink_electric_gripper side="${side}"
+                                  l_finger="$(arg l_finger)"
+                                  l_finger_slot="$(arg l_finger_slot)"
+                                  l_finger_tip="$(arg l_finger_tip)"
+                                  l_finger_grasp="$(arg l_finger_grasp)"
+                                  r_finger="$(arg r_finger)"
+                                  r_finger_slot="$(arg r_finger_slot)"
+                                  r_finger_tip="$(arg r_finger_tip)"
+                                  r_finger_grasp="$(arg r_finger_grasp)"/>
+  </xacro:if>
+  <xacro:if value="${'$(arg end_effector_type)' == 'pneumatic_gripper'}">
+    <!-- Left Pneumatic Gripper -->
+    <xacro:include filename="$(find rethink_ee_description)/urdf/pneumatic_gripper/rethink_pneumatic_gripper.xacro"/>
+    <xacro:rethink_pneumatic_gripper side="left"/>
+  </xacro:if>
+  <xacro:if value="${'$(arg end_effector_type)' not in ['electric_gripper', 'pneumatic_gripper']}">
+    <!-- Left Null Gripper -->
+    <xacro:include filename="$(find rethink_ee_description)/urdf/null_gripper/null_gripper.xacro"/>
+    <xacro:null_gripper side="left"/>
+  </xacro:if>
 </robot>

File: baxter_description/urdf/right_end_effector.urdf.xacro (robot description, xacro)
@@ -1,13 +1,37 @@
 <?xml version="1.0" ?>
 <robot name="right_end_effector" xmlns:xacro="http://www.ros.org/wiki/xacro">
-  <xacro:include filename="$(find rethink_ee_description)/urdf/electric_gripper/rethink_electric_gripper.xacro" />
-  <xacro:rethink_electric_gripper side="right"
-                                  l_finger="extended_narrow"
-                                  l_finger_slot="2"
-                                  l_finger_tip="half_round_tip"
-                                  l_finger_grasp="inner"
-                                  r_finger="extended_narrow"
-                                  r_finger_slot="2"
-                                  r_finger_tip="half_round_tip"
-                                  r_finger_grasp="inner"/>
+  <xacro:property name="side" value="right" scope="local"/>
+  <xacro:arg name="end_effector_type" default="electric_gripper"/>
+  <xacro:arg name="gazebo"            default="false"/>
+  <xacro:if value="${'$(arg end_effector_type)' == 'electric_gripper'}">
+    <!-- Left Electric Gripper -->
+    <xacro:arg name="l_finger"        default="extended_narrow"/>
+    <xacro:arg name="l_finger_slot"   default="2"/>
+    <xacro:arg name="l_finger_tip"    default="half_round_tip"/>
+    <xacro:arg name="l_finger_grasp"  default="inner"/>
+    <xacro:arg name="r_finger"        default="extended_narrow"/>
+    <xacro:arg name="r_finger_slot"   default="2"/>
+    <xacro:arg name="r_finger_tip"    default="half_round_tip"/>
+    <xacro:arg name="r_finger_grasp"  default="inner"/>
+    <xacro:include filename="$(find rethink_ee_description)/urdf/electric_gripper/rethink_electric_gripper.xacro"/>
+    <xacro:rethink_electric_gripper side="${side}"
+                                  l_finger="$(arg l_finger)"
+                                  l_finger_slot="$(arg l_finger_slot)"
+                                  l_finger_tip="$(arg l_finger_tip)"
+                                  l_finger_grasp="$(arg l_finger_grasp)"
+                                  r_finger="$(arg r_finger)"
+                                  r_finger_slot="$(arg r_finger_slot)"
+                                  r_finger_tip="$(arg r_finger_tip)"
+                                  r_finger_grasp="$(arg r_finger_grasp)"/>
+  </xacro:if>
+  <xacro:if value="${'$(arg end_effector_type)' == 'pneumatic_gripper'}">
+    <!-- Left Pneumatic Gripper -->
+    <xacro:include filename="$(find rethink_ee_description)/urdf/pneumatic_gripper/rethink_pneumatic_gripper.xacro"/>
+    <xacro:rethink_pneumatic_gripper side="right"/>
+  </xacro:if>
+  <xacro:if value="${'$(arg end_effector_type)' not in ['electric_gripper', 'pneumatic_gripper']}">
+    <!-- Left Null Gripper -->
+    <xacro:include filename="$(find rethink_ee_description)/urdf/null_gripper/null_gripper.xacro"/>
+    <xacro:null_gripper side="right"/>
+  </xacro:if>
 </robot>

Commit message: Polished URDF Xacros
- Made pedestal an optional argument (to be used with mobile bases)
- Renamed baxter_base.xacro to baxter_base.urdf.xacro to be consistent
- Made sure every mass was at least 0.0001 for Gazebo

File: baxter_description/urdf/baxter.urdf.xacro (robot description, xacro)
@@ -2,12 +2,15 @@
 <robot name="baxter" xmlns:xacro="http://www.ros.org/wiki/xacro">
   <xacro:arg name="gazebo" default="false"/>
+  <xacro:arg name="pedestal" default="true"/>
   <!-- Baxter Base URDF -->
-  <xacro:include filename="$(find baxter_description)/urdf/baxter_base/baxter_base.xacro">
+  <xacro:include filename="$(find baxter_description)/urdf/baxter_base/baxter_base.urdf.xacro">
     <xacro:arg name="gazebo" value="${gazebo}"/>
   </xacro:include>
   <!-- Baxter Pedestal -->
-  <xacro:include filename="$(find baxter_description)/urdf/pedestal/pedestal.xacro">
-    <xacro:arg name="gazebo" value="${gazebo}"/>
-  </xacro:include>
+  <xacro:if value="$(arg pedestal)">
+    <xacro:include filename="$(find baxter_description)/urdf/pedestal/pedestal.xacro">
+      <xacro:arg name="gazebo" value="${gazebo}"/>
+    </xacro:include>
+  </xacro:if>
   <!-- Left End Effector -->
   <xacro:include filename="$(find baxter_description)/urdf/left_end_effector.urdf.xacro" />

File: rethink_ee_description/urdf/electric_gripper/rethink_electric_gripper.xacro (robot description, xacro)
@@ -53,5 +53,5 @@
       <inertial>
         <origin rpy="0 0 0" xyz="0 0 0"/>
-        <mass value="0.0"/>
+        <mass value="0.0001"/>
         <inertia ixx="0" ixy="0" ixz="0" iyy="0" iyz="0" izz="0.0"/>
       </inertial>

File: rethink_ee_description/urdf/pneumatic_gripper/pneumatic_gripper_base.xacro (robot description, xacro)
@@ -43,5 +43,5 @@
       <inertial>
         <origin rpy="0 0 0" xyz="0 0 0"/>
-        <mass value="0.0"/>
+        <mass value="0.0001"/>
         <inertia ixx="0" ixy="0" ixz="0" iyy="0" iyz="0" izz="0.0"/>
       </inertial>

File: rethink_ee_description/urdf/pneumatic_gripper/rethink_pneumatic_gripper.xacro (robot description, xacro)
@@ -42,5 +42,5 @@
       <inertial>
         <origin rpy="0 0 0" xyz="0 0 0"/>
-        <mass value="0.0"/>
+        <mass value="0.0001"/>
         <inertia ixx="0" ixy="0" ixz="0" iyy="0" iyz="0" izz="0.0"/>
       </inertial>
